Commit message: added 3D lidar and pc processing node

File: robot_description/urdf/robot.gazebo.xacro (robot description, xacro)
@@ -92,5 +92,5 @@
     </plugin>
   </gazebo>
-  <gazebo reference="base_scan">
+  <!--<gazebo reference="base_scan">
     <material>Gazebo/FlatBlack</material>
     <sensor type="ray" name="lds_lfcd_sensor">
@@ -123,4 +123,4 @@
       </plugin>
     </sensor>
-  </gazebo>
+  </gazebo> -->
 </robot>

File: robot_description/urdf/robot.urdf.xacro (robot description, xacro)
@@ -113,5 +113,5 @@
   </joint>
   <link name="imu_link"/>
-  <joint name="scan_joint" type="fixed">
+  <!--<joint name="scan_joint" type="fixed">
     <parent link="base_link"/>
     <child link="base_scan"/>
@@ -139,6 +139,6 @@
                izz="0.001" />
     </inertial>
-  </link>
-  <!-- Remove after you create new file. Do not want to change the source code-->
+  </link> -->
+  <!-- Remove after you create new file. Do not want to change the source code
   <xacro:include filename="$(find kinect_description)/urdf/kinect/kinect.xacro">
         <xacro:arg name="gazebo" value="${gazebo}"/>
@@ -152,4 +152,12 @@
                          cam_or="0.0"
                          cam_op="${pi/180}"
-                         cam_oy="0.3"/>
+                         cam_oy="0.3"/> -->
+  <xacro:arg name="gpu" default="false"/>
+  <xacro:property name="gpu" value="$(arg gpu)" />
+  <xacro:arg name="organize_cloud" default="false"/>
+  <xacro:property name="organize_cloud" value="$(arg organize_cloud)" />
+  <xacro:include filename="$(find velodyne_description)/urdf/VLP-16.urdf.xacro"/>
+  <xacro:VLP-16 parent="base_link" name="velodyne" topic="/velodyne_points" organize_cloud="${organize_cloud}" hz="10" samples="440" gpu="${gpu}">
+    <origin xyz="-0.025 0 0.145" rpy="0 0 0" />
+  </xacro:VLP-16>
 </robot>
